File: eagle/solderstation_v1_6.sch (EAGLE design)
At the start: 41 parts, among them IC1 OPA336U, IC2 78L05F, J1 POWER_JACKPTH, T1 IRF7416, T2 BSN20, T3 BSN20

Commit message: update with schematic
Other:
- note added: "MW"
- note added: "Matthias Wagner"
- note added: "http://debugginglab.wordpress.com"
Changed lines of the file:
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@@
 <?xml version="1.0" encoding="utf-8"?>
 <!DOCTYPE eagle SYSTEM "eagle.dtd">
-<eagle version="6.5.0">
+<eagle version="6.1">
 <drawing>
 <settings>
@@
 <wire x1="330.2" y1="50.8" x2="330.2" y2="91.44" width="0.6096" layer="94"/>
 <text x="334.518" y="81.534" size="3.81" layer="94" ratio="14">Display</text>
+<text x="289.56" y="5.08" size="1.778" layer="91">http://debugginglab.wordpress.com</text>
+<text x="289.56" y="15.24" size="6.4516" layer="91">MW</text>
+<text x="289.56" y="12.7" size="1.4224" layer="91">Matthias Wagner</text>
 </plain>
 <instances>
